File: MechKBNumpad1/MechKBNumpad1(STM32Version).sch (KiCad schematic (older format))
At the start: 51 parts, among them J1 TYPE-C-31-M12_13-acheronSymbo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, J2 Conn_ARM_JTAG_SWD_10, Q1 DTC123J, SW1 SW_Push, U1 ATmega32U4-AU, U1 STM32F072-LQFP48-acheronSymbo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, U2 USBLC6-2SC6-Power_Protection, U3 MCP1700-3302E_SOT23, Y1 Crystal_GND24_Small

Commit message: Add files via upload
Parts:
- removed C1, C2, C7: 4.7u, Capacitor_SMD:C_0805_2012Metric_Pad1.18x1.45mm_HandSolder, symbol Device:C_Small
- removed C3, C4, C5, C6: 0.1u, Capacitor_SMD:C_0805_2012Metric_Pad1.18x1.45mm_HandSolder, symbol Device:C_Small
- removed C8: 1u, Diode_SMD:D_SOD-123, symbol Device:C_Small
- removed ESD1: PRTR5V0U2X, Package_TO_SOT_SMD:SOT-143, symbol Power_Protection:PRTR5V0U2X
- removed F1: 500mA, Fuse:Fuse_1206_3216Metric_Pad1.42x1.75mm_HandSolder, symbol Device:Polyfuse_Small
- removed R1: 10k, Resistor_SMD:R_0805_2012Metric_Pad1.20x1.40mm_HandSolder, symbol Device:R
- removed R2: 10K, Resistor_SMD:R_0805_2012Metric_Pad1.20x1.40mm_HandSolder, symbol Device:R_Small
- removed R3, R4, R5, R6: 22, Resistor_SMD:R_0805_2012Metric_Pad1.20x1.40mm_HandSolder, symbol Device:R_Small
- removed R7, R8: 5.1K, Resistor_SMD:R_0805_2012Metric_Pad1.20x1.40mm_HandSolder, symbol Device:R_Small
- removed SW1: SW_Push, Button_Switch_SMD:SW_SPST_SKQG_WithStem, symbol Switch:SW_Push
- removed U1: ATmega32U4-AU, Package_QFP:TQFP-44_10x10mm_P0.8mm, symbol MCU_Microchip_ATmega:ATmega32U4-AU
- removed USB1: HRO-TYPE-C-31-M-12, type_c:HRO-TYPE-C-31-M-12-HandSoldering, symbol USB_C:HRO-TYPE-C-31-M-12
- removed Y1: Crystal_GND24_Small, Crystal:Crystal_SMD_3225-4Pin_3.2x2.5mm_HandSoldering, symbol Device:Crystal_GND24_Small
Connections:
- no-connect marks 4 -> 2
