File: MechKBNumpad1/MechKBNumpad1.kicad_pcb (KiCad board)
At the start: 2 copper layers, 76 parts, among them SW1 SW_Push, U1 ATmega32U4-AU, Y1 Crystal_GND24_Small

Commit message: Add files via upload
Parts:
- moved MX1 7.78 mm to (53.2, 61.0)
- moved MX2 7.78 mm to (72.2, 61.0)
- moved MX3 7.78 mm to (91.3, 61.0)
- moved MX4 7.78 mm to (110.3, 61.0)
