File: MechKBNumpad1/MechKBNumpad1.sch (KiCad schematic (older format))
At the start: 22 parts, among them SW1 SW_Push, U1 ATmega32U4-AU, Y1 Crystal_GND24_Small

Commit message: Add files via upload
Parts:
- added CB1, CSO1: 1uF, Capacitor_SMD:C_0805_2012Metric_Pad1.18x1.45mm_HandSolder, symbol Device:C_Small
- added CB2: 10nF, Capacitor_SMD:C_0805_2012Metric_Pad1.18x1.45mm_HandSolder, symbol Device:C_Small
- added CB3, CB5, CB7, CB8: 100n, Capacitor_SMD:C_0805_2012Metric_Pad1.18x1.45mm_HandSolder, symbol Device:C_Small
- added CB4, CB6: 4.7u, Capacitor_SMD:C_0805_2012Metric_Pad1.18x1.45mm_HandSolder, symbol Device:C_Small
- added CRST1, CRST2: 4.7nF, Capacitor_SMD:C_0805_2012Metric_Pad1.18x1.45mm_HandSolder, symbol Device:C_Small
- added CSH1: 4.7uF, Capacitor_SMD:C_0805_2012Metric_Pad1.18x1.45mm_HandSolder, symbol Device:C_Small
- added CSI1: 10uF, Capacitor_SMD:C_0805_2012Metric_Pad1.18x1.45mm_HandSolder, symbol Device:C_Small
- added D?: 1N4007, Diode_THT:D_DO-41_SOD81_P10.16mm_Horizontal, symbol Diode:1N4007
- added DF1: RB060m-60TR, symbol Device:D_Schottky
- added DRST1: 1N4148, Diode_THT:D_DO-35_SOD27_P7.62mm_Horizontal, symbol Diode:1N4148
- added F1: Polyfuse, symbol Device:Polyfuse
- added J1: TYPE-C-31-M12_13-acheronSymbols, acheronConnectors:TYPE-C-31-M-12, symbol Hammerhead_rescue:TYPE-C-31-M12_13-acheronSymbols
- added J2: Conn_ARM_JTAG_SWD_10, symbol Connector:Conn_ARM_JTAG_SWD_10
- added Q1: DTC123J, symbol Transistor_BJT:DTC123J
- added RCC1, RCC2: 5.1K, Resistor_SMD:R_0805_2012Metric_Pad1.20x1.40mm_HandSolder, symbol Device:R_Small
- added RF1: 10K, Resistor_SMD:R_0805_2012Metric_Pad1.20x1.40mm_HandSolder, symbol Device:R_Small
- added RRST1: 100K, Resistor_SMD:R_0805_2012Metric_Pad1.20x1.40mm_HandSolder, symbol Device:R_Small
- added RSH1: 1M, Resistor_SMD:R_0805_2012Metric_Pad1.20x1.40mm_HandSolder, symbol Device:R_Small
- added SW1: SW_Push, Button_Switch_SMD:SW_SPST_SKQG_WithStem, symbol Switch:SW_Push
- added U1: STM32F072-LQFP48-acheronSymbols, acheron_Components:TQPF-44_10x10mm_P0.8mm, symbol Hammerhead_rescue:STM32F072-LQFP48-acheronSymbols
- added U2: USBLC6-2SC6-Power_Protection, Package_TO_SOT_SMD:SOT-23-6, symbol Hammerhead_rescue:USBLC6-2SC6-Power_Protection
- added U3: MCP1700-3302E_SOT23, Package_TO_SOT_SMD:SOT-23, symbol Hammerhead_cache:MCP1700-3302E_SOT23
Connections:
- net D+: now also U1.33 (USB_DP/PA12), U2.3 (IO2)
- net D-: now also U1.32 (USB_DM/TIM1_CH4/PA11), U2.1 (IO1)
- net GND: now also CB1.2, CB2.2, CB3.2, CB4.2, CB5.2, CB6.2, CB7.1, CB8.2, CRST1.1, CRST2.2, CSH1.1, CSI1.2, CSO1.2, DF1.2 (A), J1.A1 (GND), J1.B1 (GND), J2.3 (GND), J2.5 (GND), J2.9 (GNDDetect), Q1.2 (E), RCC1.2, RCC2.1, RF1.2, RRST1.1, RSH1.2, U1.23 (VSS), U1.35 (VSS), U1.47 (VSS), U1.8 (VSSA), U2.2 (GND), U3.1 (GND)
- new net: DRST1.2 (A), Q1.1 (B), SW1.2
- new net: J1.A5 (CC1), RCC1.1
- new net: J1.B5 (CC2), RCC2.2
- new net: CSH1.2, J1.S (SHIELD), RSH1.1
- new net 3.3V: CB1.1, CB2.1, CB3.1, CB4.1, CB5.1, CB6.1, CB7.2, CB8.1, CSO1.1, D?.2 (A), J2.1 (VTref), SW1.1, U1.1 (VBAT), U1.24 (VDD), U1.36 (VDDIO2), U1.48 (VDD), U1.9 (VDDA), U3.2 (VO)
- new net 5V: CSI1.1, D?.1 (K), DF1.1 (K), F1.1, RF1.1, U3.3 (VI)
- new net BOOT0: CRST1.2, DRST1.1 (K), RRST1.2, U1.44 (BOOT0)
- new net DBUS+: J1.A7 (D-), J1.B7 (D-), U2.4 (IO2)
- new net DBUS-: J1.A6 (D+), J1.B6 (D+), U2.6 (IO1)
- new net NRST: CRST2.1, J2.10 (~RESET~), Q1.3 (C), U1.7 (NRST)
- new net SWCLK: J2.4 (SWDCLK/TCK), U1.37 (SWCLK/PA14)
- new net SWDIO: J2.2 (SWDIO/TMS), U1.34 (SWDIO/PA13)
- new net VBUS: F1.2, J1.A4 (VBUS), J1.B4 (VBUS), U2.5 (VBUS)
- no-connect marks 2 -> 4
Other:
- moved on the sheet: C1, C2, C3, C4, C5, C6, C7, C8, ESD1, F1, R1, R2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
