File: MechKBNumpad1/SwitchMatrix.sch (KiCad schematic (older format))
At the start: 54 parts

Commit message: Add files via upload
Parts:
- removed D10: D, Diode_SMD:D_SOD-123, symbol Device:D
- removed MX10: mute, MX_Alps_keys:MX-1U-NoLED, symbol MX_Alps:MX-NoLED
- removed MX5: encoder, MX_Alps_keys:MX-1U-NoLED, symbol MX_Alps:MX-NoLED
- added C1, C2: C_Small, symbol Device:C_Small
- added SW1: Rotary_Encoder_Switch, symbol Device:Rotary_Encoder_Switch
- MX14: value macro1 -> mute
- MX19: value macro2 -> macro1
- MX23: value macro3 -> macro2
- MX27: value macro4 -> macro3
Connections:
- net labels added: power_GND
- wire segments 65 -> 79
Changed lines of the file:
@@
 Connection ~ 4900 4350
-$Comp
-L MX_Alps:MX-NoLED MX5
-U 1 1 60FD148D
-P 6100 1250
-F 0 "MX5" H 6133 1473 60  0000 C CNN
-F 1 "encoder" H 6133 1399 20  0000 C CNN
-F 2 "MX_Alps_keys:MX-1U-NoLED" H 5475 1225 60  0001 C CNN
-F 3 "" H 5475 1225 60  0001 C CNN
-	1    6100 1250
-	1    0    0    -1
-$EndComp
 $Comp
 L Device:D D?
@@
 	6050 1700 6550 1700
 Connection ~ 6050 1700
-Wire Wire Line
-	6250 1200 6250 850
-Connection ~ 6250 1200
-$Comp
-L MX_Alps:MX-NoLED MX10
-U 1 1 60FD14B6
-P 6100 2300
-F 0 "MX10" H 6133 2523 60  0000 C CNN
-F 1 "mute" H 6133 2449 20  0000 C CNN
-F 2 "MX_Alps_keys:MX-1U-NoLED" H 5475 2275 60  0001 C CNN
-F 3 "" H 5475 2275 60  0001 C CNN
-	1    6100 2300
-	1    0    0    -1
-$EndComp
-$Comp
-L Device:D D?
-U 1 1 60FD14C0
-P 6050 2600
-AR Path="/60FD14C0" Ref="D?"  Part="1"
-AR Path="/60F1F468/60FD14C0" Ref="D10"  Part="1"
-F 0 "D10" V 6096 2520 50  0000 R CNN
-F 1 "D" V 6005 2520 50  0000 R CNN
-F 2 "Diode_SMD:D_SOD-123" H 6050 2600 50  0001 C CNN
-F 3 "~" H 6050 2600 50  0001 C CNN
-	1    6050 2600
-	0    -1   -1   0
-$EndComp
-Wire Wire Line
-	6050 2750 6550 2750
-Connection ~ 6050 2750
-Connection ~ 6250 2250
-Wire Wire Line
-	6250 1200 6250 2250
 $Comp
 L MX_Alps:MX-NoLED MX14
@@
 P 6100 3350
 F 0 "MX14" H 6133 3573 60  0000 C CNN
-F 1 "macro1" H 6133 3499 20  0000 C CNN
+F 1 "mute" H 6133 3499 20  0000 C CNN
 F 2 "MX_Alps_keys:MX-1U-NoLED" H 5475 3325 60  0001 C CNN
 F 3 "" H 5475 3325 60  0001 C CNN
@@
 P 6100 4400
 F 0 "MX19" H 6133 4623 60  0000 C CNN
-F 1 "macro2" H 6133 4549 20  0000 C CNN
+F 1 "macro1" H 6133 4549 20  0000 C CNN
 F 2 "MX_Alps_keys:MX-1U-NoLED" H 5475 4375 60  0001 C CNN
 F 3 "" H 5475 4375 60  0001 C CNN
@@
 Wire Wire Line
 	6250 3300 6250 4350
-Wire Wire Line
-	6250 2250 6250 3300
 $Comp
 L MX_Alps:MX-NoLED MX23
@@
 P 6100 5500
 F 0 "MX23" H 6133 5723 60  0000 C CNN
-F 1 "macro3" H 6133 5649 20  0000 C CNN
+F 1 "macro2" H 6133 5649 20  0000 C CNN
 F 2 "MX_Alps_keys:MX-1U-NoLED" H 5475 5475 60  0001 C CNN
 F 3 "" H 5475 5475 60  0001 C CNN
@@
 P 6100 6550
 F 0 "MX27" H 6133 6773 60  0000 C CNN
-F 1 "macro4" H 6133 6699 20  0000 C CNN
+F 1 "macro3" H 6133 6699 20  0000 C CNN
 F 2 "MX_Alps_keys:MX-1U-NoLED" H 5475 6525 60  0001 C CNN
 F 3 "" H 5475 6525 60  0001 C CNN
@@
 Wire Wire Line
 	4700 1700 6050 1700
-Wire Wire Line
-	4700 2750 6050 2750
 Wire Wire Line
 	4700 4850 6050 4850
@@
 Text GLabel 6250 850  1    50   Input ~ 0
 col4
+Wire Wire Line
+	4700 2750 6550 2750
+$Comp
+L Device:Rotary_Encoder_Switch SW1
+U 1 1 60E8B9FD
+P 6700 1250
+F 0 "SW1" H 6700 883 50  0000 C CNN
+F 1 "Rotary_Encoder_Switch" H 6700 974 50  0000 C CNN
+F 2 "" H 6550 1410 50  0001 C CNN
+F 3 "~" H 6700 1510 50  0001 C CNN
+	1    6700 1250
+	-1   0    0    1
+$EndComp
+Wire Wire Line
+	6400 1350 6050 1350
+Wire Wire Line
+	6050 1350 6050 1400
+Wire Wire Line
+	6400 1150 6250 1150
+Wire Wire Line
+	6250 850  6250 1150
+Connection ~ 6250 1150
+Wire Wire Line
+	6250 1150 6250 3300
+$Comp
+L voyager20cahce:power_GND #PWR01
+U 1 1 60E8FC10
+P 8100 1300
+F 0 "#PWR01" H 8100 1050 50  0001 C CNN
+F 1 "power_GND" H 8105 1127 50  0000 C CNN
+F 2 "" H 8100 1300 50  0001 C CNN
+F 3 "" H 8100 1300 50  0001 C CNN
+	1    8100 1300
+	1    0    0    -1
+$EndComp
+Wire Wire Line
+	7000 1250 7600 1250
+Wire Wire Line
+	8100 1250 8100 1300
+$Comp
+L Device:C_Small C2
+U 1 1 60E92032
+P 7600 1350
+F 0 "C2" H 7692 1396 50  0000 L CNN
+F 1 "C_Small" H 7692 1305 50  0000 L CNN
+F 2 "" H 7600 1350 50  0001 C CNN
+F 3 "~" H 7600 1350 50  0001 C CNN
+	1    7600 1350
+	1    0    0    -1
+$EndComp
+Connection ~ 7600 1250
+Wire Wire Line
+	7600 1250 8100 1250
+$Comp
+L Device:C_Small C1
+U 1 1 60E92C9F
+P 7600 1150
+F 0 "C1" H 7692 1196 50  0000 L CNN
+F 1 "C_Small" H 7692 1105 50  0000 L CNN
+F 2 "" H 7600 1150 50  0001 C CNN
+F 3 "~" H 7600 1150 50  0001 C CNN
+	1    7600 1150
+	1    0    0    -1
+$EndComp
+Wire Wire Line
+	7000 1150 7300 1150
+Wire Wire Line
+	7300 1150 7300 1050
+Wire Wire Line
+	7300 1050 7600 1050
+Wire Wire Line
+	7000 1350 7300 1350
+Wire Wire Line
+	7300 1350 7300 1450
+Wire Wire Line
+	7300 1450 7600 1450
+Wire Wire Line
+	7600 1050 8100 1050
+Wire Wire Line
+	8100 1050 8100 1000
+Connection ~ 7600 1050
+Wire Wire Line
+	7600 1450 7850 1450
+Wire Wire Line
+	7850 1450 7850 1700
+Connection ~ 7600 1450
 $EndSCHEMATC
